File: MCU.kicad_sch (KiCad schematic)
At the start: 18 parts, among them J1 USB_C_Receptacle_USB2.0_14P, SW1 SW_Push, U4 ESP32-S3-WROOM-1

Commit message: Ethernet W55000 controller added
Parts:
- added R26, R54: 10k, Resistor_SMD:R_0805_2012Metric, symbol Device:R
Connections:
- net +3V3: now also R26.1, R54.1
- net I2C.SCL: now also R26.2
- net I2C.SDA: now also R54.2
