File: StairsV2Eth_MainBoard/Power.kicad_sch (KiCad schematic)
At the start: 26 parts, among them J5 Conn_01x02, U5 TPS62933, U6 AMS1117-3.3

Commit message: Mainvoard PCB Added
Parts:
- removed C7: 10, Capacitor_SMD:C_0805_2012Metric, symbol Device:C
- removed J5: Conn_01x02, TerminalBlock_Phoenix:TerminalBlock_Phoenix_PT-1,5-2-5.0-H_1x02_P5.00mm_Horizontal, symbol Connector_Generic:Conn_01x02
- added C7, C8: 47u 10V, Capacitor_SMD:CP_Elec_5x5.4, symbol Device:C_Polarized
- added J16: Conn_01x04, Connector_Phoenix_MC:PhoenixContact_MCV_1,5_4-G-3.5_1x04_P3.50mm_Vertical, symbol Connector_Generic:Conn_01x04
- C9: renamed from C34; value 10 -> 0.1
- renumbered C6 to C1, C7 to C2, C31 to C3, C32 to C4, C33 to C5, L2 to L1, R19 to R2, R20 to R3, R2 to R4, R1 to R5, R2 to R6, R5 to R7, R6 to R8, U5 to U1, U6 to U2
Connections:
- net +24V: now also C1.1, C2.1, D1.1 (K), R1.1, R2.1, U1.3 (VIN); no longer D1.2 (A)
- net +3V3: now also C8.1
- net +5V: now also C7.1
- net GND: now also C7.2, C8.2, J16.4 (Pin_4)
- new net Earth_Protective: J16.1 (Pin_1)
- new net VIN: D1.2 (A), J16.2 (Pin_2), J16.3 (Pin_3)
Other:
- moved on the sheet: C1, C2, C3, C4, C5, C6, C9, D1, D2, L1, R1, R2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
